File: LM1876_mute.kicad_pcb (KiCad board)
At the start: 2 copper layers, 22.5 x 14.2 mm, 11 parts, among them J3 POWER_HEADER, J4 MUTE_HEADER, J5 STBY, Q1 2N7002

Commit message: added imgs
Other:
- board text added: "GND"
- board text added: "MUTE"
- board text added: "V+"
